Commit message: no more stl meshes for simplicity

File: robots/nori/so101_new_calib.urdf (robot description, URDF)
Before this commit: robot so101_new_calib, 8 links, 7 joints
Links:
- link base_link: geometry 
- link gripper_link: geometry 
- link lower_arm_link: geometry 
- link moving_jaw_so101_v1_link: geometry 
- link shoulder_link: geometry 
- link upper_arm_link: geometry 
- link wrist_link: geometry 
